Commit message: added rtabmap database file

File: my_robot/urdf/my_robot.xacro (robot description, xacro)
@@ -2,8 +2,10 @@
 <robot name="my_robot" xmlns:xacro="http://www.ros.org/wiki/xacro">
   <xacro:include filename="$(find my_robot)/urdf/my_robot.gazebo" />
-  <!-- Robot Footprint Link -->
-  <link name="robot_footprint">
-  </link>
-  <!-- Chassis Link -->
+  <link name="robot_footprint"></link>
+  <joint name="robot_footprint_joint" type="fixed">
+    <origin xyz="0 0 0" rpy="0 0 0" />
+    <parent link="robot_footprint"/>
+    <child link="chassis" />
+  </joint>
   <link name='chassis'>
     <pose>0 0 0.1 0 0 0</pose>
@@ -12,11 +14,10 @@
       <origin xyz="0.0 0 0" rpy=" 0 0 0"/>
       <inertia
-          ixx="0.1" ixy="0" ixz="0"
-          iyy="0.1" iyz="0"
-          izz="0.1"
+              ixx="0.1" ixy="0" ixz="0"
+              iyy="0.1" iyz="0"
+              izz="0.1"
       />
     </inertial>
-    <!-- Chassis Collision & Visual -->
-    <collision name='chassis_collision'>
+    <collision name='collision'>
       <origin xyz="0 0 0" rpy=" 0 0 0"/>
       <geometry>
@@ -30,5 +31,4 @@
       </geometry>
     </visual>
-    <!-- Back Caster Collision & Visual -->
     <collision name='back_caster_collision'>
       <origin xyz="-0.15 0 -0.05" rpy=" 0 0 0"/>
@@ -43,5 +43,4 @@
       </geometry>
     </visual>
-    <!-- Front Caster Collision & Visual -->
     <collision name='front_caster_collision'>
       <origin xyz="0.15 0 -0.05" rpy=" 0 0 0"/>
@@ -57,21 +56,20 @@
     </visual>
   </link>
-  <!-- Joint Between Robot Footprint & Chassis -->
-  <joint name="robot_footprint_joint" type="fixed">
-    <origin xyz="0 0 0" rpy="0 0 0" />
-    <parent link="robot_footprint"/>
-    <child link="chassis" />
-  </joint>
-  <!-- Left Wheel Link -->
-  <link name='left_wheel'>
+  <!-- Add two wheels -->
+  <link name="left_wheel">
     <inertial>
-    <origin xyz="0 0 0" rpy="0 1.5707 1.5707"/>
-    <mass value="5"/>
+      <origin xyz="0 0 0" rpy="0 1.5707 1.5707"/>
+      <mass value="5"/>
       <inertia
-          ixx="0.1" ixy="0" ixz="0"
-          iyy="0.1" iyz="0"
-          izz="0.1"
+              ixx="0.1" ixy="0" ixz="0"
+              iyy="0.1" iyz="0" izz="0.1"
       />
     </inertial>
+    <collision>
+      <origin xyz="0 0 0" rpy="0 1.5707 1.5707"/>
+      <geometry>
+        <cylinder radius="0.1" length="0.05"/>
+      </geometry>
+    </collision>
     <visual>
       <origin xyz="0 0 0" rpy="0 1.5707 1.5707"/>
@@ -80,4 +78,14 @@
       </geometry>
     </visual>
+  </link>
+  <link name="right_wheel">
+    <inertial>
+      <origin xyz="0 0 0" rpy="0 1.5707 1.5707"/>
+      <mass value="5"/>
+      <inertia
+              ixx="0.1" ixy="0" ixz="0"
+              iyy="0.1" iyz="0" izz="0.1"
+      />
+    </inertial>
     <collision>
       <origin xyz="0 0 0" rpy="0 1.5707 1.5707"/>
@@ -86,56 +94,38 @@
       </geometry>
     </collision>
+    <visual>
+      <origin xyz="0 0 0" rpy="0 1.5707 1.5707"/>
+      <geometry>
+        <cylinder radius="0.1" length="0.05"/>
+      </geometry>
+    </visual>
   </link>
-  <!-- Joint Between Chassis & Left Wheel -->
   <joint name="left_wheel_hinge" type="continuous">
-    <origin xyz="0 0.15 0" rpy="0 0 0" />
+    <origin xyz="0 0.125 0" rpy="0 0 0"/>
+    <child link="left_wheel"/>
     <parent link="chassis"/>
-    <child link="left_wheel" />
     <axis xyz="0 1 0" rpy="0 0 0"/>
     <limit effort="10000" velocity="1000"/>
     <dynamics damping="1.0" friction="1.0"/>
   </joint>
-  <!-- Right Wheel Link -->
-  <link name='right_wheel'>
-    <inertial>
-    <origin xyz="0 -0.3 0" rpy="0 1.5707 1.5707"/>
-    <mass value="5"/>
-      <inertia
-          ixx="0.1" ixy="0" ixz="0"
-          iyy="0.1" iyz="0"
-          izz="0.1"
-      />
-    </inertial>
-    <visual>
-      <origin xyz="0 -0.3 0" rpy="0 1.5707 1.5707"/>
-      <geometry>
-        <cylinder radius="0.1" length="0.05"/>
-      </geometry>
-    </visual>
-    <collision>
-      <origin xyz="0 -0.3 0" rpy="0 1.5707 1.5707"/>
-      <geometry>
-        <cylinder radius="0.1" length="0.05"/>
-      </geometry>
-    </collision>
-  </link>
-  <!-- Joint Between Chassis & Right Wheel -->
   <joint name="right_wheel_hinge" type="continuous">
-    <origin xyz="0 0.15 0" rpy="0 0 0" />
+    <origin xyz="0 -0.125 0" rpy="0 0 0"/>
+    <child link="right_wheel"/>
     <parent link="chassis"/>
-    <child link="right_wheel" />
     <axis xyz="0 1 0" rpy="0 0 0"/>
     <limit effort="10000" velocity="1000"/>
     <dynamics damping="1.0" friction="1.0"/>
   </joint>
-  <!-- Camera Link -->
-  <link name="camera_link">
+  <!-- Add camera -->
+  <link name="camera">
+    <origin xyz="0 0 0" rpy="0 0 0" />
     <inertial>
-      <origin xyz="0 0 0" rpy="0 0 0"/>
       <mass value="0.1"/>
-      <inertia ixx="1e-6" ixy="0" ixz="0.0" iyy="1e-6" iyz="0" izz="1e-6"/>
+      <inertia
+              ixx="1e-6" ixy="0" ixz="0"
+              iyy="1e-6" iyz="0" izz="1e-6"
+      />
     </inertial>
     <collision>
-      <origin xyz="0 0 0" rpy="0 0 0"/>
       <geometry>
         <box size="0.05 0.05 0.05"/>
@@ -143,5 +133,4 @@
     </collision>
     <visual>
-      <origin xyz="0 0 0" rpy="0 0 0"/>
       <geometry>
         <box size="0.05 0.05 0.05"/>
@@ -149,35 +138,34 @@
     </visual>
   </link>
-  <!-- Joint Between Chassis & Camera Link -->
   <joint name="camera_joint" type="fixed">
-    <origin xyz="0.2 0.0 0.0" rpy="0.0 0.0 0.0"/>
+    <axis xyz="0 1 0"/>
+    <origin xyz="0.2 0 0" rpy="0 0 0" />
     <parent link="chassis"/>
-    <child link="camera_link"/>
-    <axis xyz="0.0 1.0 0.0"/>
+    <child link="camera" />
   </joint>
-  <!-- Optical Camera Link -->
+  <!-- Add RGB-D camera -->
+  <joint name="camera_optical_joint" type="fixed">
+    <origin xyz="0 0 0" rpy="-1.5707 0 -1.5707"/>
+    <parent link="camera"/>
+    <child link="camera_link_optical"/>
+  </joint>
   <link name="camera_link_optical">
   </link>
-  <!-- Joint Between Camera & Optical Camera Link -->
-  <joint name="camera_optical_joint" type="fixed">
-    <origin xyz="0 0 0" rpy="-1.5707 0 -1.5707"/>
-    <parent link="camera_link"/>
-    <child link="camera_link_optical"/>
-  </joint>
-  <!-- Lidar Link -->
+  <!-- Add Lidar -->
   <link name="hokuyo">
+    <origin xyz="0 0 0" rpy="0 0 0" />
     <inertial>
-      <origin xyz="0 0 0" rpy="0 0 0"/>
       <mass value="1e-5"/>
-      <inertia ixx="1e-6" ixy="0" ixz="0" iyy="1e-6" iyz="0" izz="1e-6"/>
+      <inertia
+              ixx="1e-6" ixy="0" ixz="0"
+              iyy="1e-6" iyz="0" izz="1e-6"
+      />
     </inertial>
     <collision>
-      <origin xyz="0 0 0" rpy="0 0 0"/>
       <geometry>
-        <box size="0.1 0.1 0.1"/>
+        <box size=".1 .1 .1"/>
       </geometry>
     </collision>
     <visual>
-      <origin xyz="0 0 0" rpy="0 0 0"/>
       <geometry>
         <mesh filename="package://my_robot/meshes/hokuyo.dae"/>
@@ -185,23 +173,22 @@
     </visual>
   </link>
-  <!-- Joint Between Chassis & Lidar -->
   <joint name="hokuyo_joint" type="fixed">
-    <origin xyz="0.15 0.0 0.1" rpy="0.0 0.0 0.0"/>
+    <axis xyz="0 1 0"/>
+    <origin xyz="0.15 0 0.1" rpy="0 0 0" />
     <parent link="chassis"/>
-    <child link="hokuyo"/>
-    <axis xyz="0.0 1.0 0.0"/>
+    <child link="hokuyo" />
   </joint>
-  <!-- Colours -->
+  <!-- Color the components -->
   <gazebo reference="chassis">
-    <material>Gazebo/Yellow</material>
+    <material>Gazebo/Orange</material>
   </gazebo>
   <gazebo reference="left_wheel">
-    <material>Gazebo/Yellow</material>
+    <material>Gazebo/Green</material>
   </gazebo>
   <gazebo reference="right_wheel">
-    <material>Gazebo/Yellow</material>
+    <material>Gazebo/Green</material>
   </gazebo>
   <gazebo reference="camera">
-    <material>Gazebo/Yellow</material>
+    <material>Gazebo/Red</material>
   </gazebo>
-</robot>
+  </robot>
